File: HW/EthernetPortX.sch (KiCad schematic (older format))
At the start: 17 parts, among them J1 RJ45_0, U12 KSZ8081MNX

Commit message: Releasing IsoSwitch.201802
Parts:
- U12: Part (none) -> KSZ8081MNXCA-TR
