File: HW/HW.kicad_pcb (KiCad board)
At the start: 4 copper layers, 62 x 49.8 mm, 131 parts, among them J1 10118193-0001LF, J10 RJ45_0, J11 RJ45_0, J12 RJ45_0, J13 RJ45_0, J2 2x10 Vertical Pin, U1 XL216-512-TQ128_CHIP_VIEW, U10 KSZ8081MNX, U11 KSZ8081MNX, U12 KSZ8081MNX, U13 KSZ8081MNX, U2 ST1S06, U3 ST1S06, U4 APX809S-46SA, U5 NCP303LSN10T, X1 DSC6001CI2A-025.0000

Commit message: Releasing IsoSwitch.201802
Parts:
- removed Mount1: , Connectors:1pin
- added J7: NWAY_TP, Measurement_Points:Measurement_Point_Square-SMD-Pad_Small, F.Cu at (149.3, 95.5)
- added J8: CRS_TP, Measurement_Points:Measurement_Point_Square-SMD-Pad_Small, F.Cu at (151.7, 95.4)
- added J9: COL_TP, Measurement_Points:Measurement_Point_Square-SMD-Pad_Small, F.Cu at (154.2, 95.4)
- C73: moved to B.Cu
- J10, J11, J12, J13: footprint TempRJ45:RJ45_8 -> RJ45_LINK-PP:RJ45_LINK-PP
- RV1: value V5.5MLA0603 -> V5.5MLA0603H
- U2, U3: footprint Housings_DFN_QFN:DFN-6-1EP_3x3mm_Pitch0.95mm -> ST1S06:DFN6D_3x3mm
- U4: value APX809S-46SA -> APX811-46UG-7; footprint TO_SOT_Packages_SMD:SOT-23 -> TO_SOT_Packages_SMD:SOT-143
- moved Mount2 16.2 mm to (170.8, 115.5)
- moved C73 1.17 mm to (143.1, 96.5), turned to 270 degrees
- moved FB121 1.07 mm to (146.9, 126.8)
- moved C121 0.98 mm to (147.7, 127.3)
- moved C82 0.66 mm to (143.9, 95.3), turned to 0 degrees
- moved U4 0.61 mm to (173.5, 104.1), turned to 180 degrees
- moved C83 0.58 mm to (147.7, 106.2)
- moved R136 0.53 mm to (169.4, 119.3)
- moved C64 0.48 mm to (141.3, 95.4)
- moved C7 0.48 mm to (122.8, 98.6), turned to 90 degrees
- moved R111 0.46 mm to (144.6, 126.2)
- moved C118 0.38 mm to (139.4, 123.3)
- moved C127 0.36 mm to (154.4, 123.0)
- moved C136 0.33 mm to (167.7, 127.2)
- moved C132 0.30 mm to (162.6, 124.0)
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Connections:
- J2 pad 15: Net-(J2-Pad15) -> COL0
- J2 pad 17: Net-(J2-Pad17) -> CRS0
- J2 pad 19: Net-(J2-Pad19) -> NWAYEN0
- U1 pad 57: /Tile0/EthernetPort0/COL -> COL0
- U1 pad 58: /Tile0/EthernetPort0/CRS -> CRS0
- U1 pad 60: /Tile0/EthernetPort0/NWAYEN -> NWAYEN0
- U10 pad 28: /Tile0/EthernetPort0/COL -> COL0
- U10 pad 29: /Tile0/EthernetPort0/CRS -> CRS0
- U10 pad 30: /Tile0/EthernetPort0/NWAYEN -> NWAYEN0
- U4 pad 3: +5V -> Net-(U4-Pad3)
Routing:
- net GND: track 348.1 -> 415.3 mm
- net +3V3: track 496.3 -> 551.0 mm, vias 51 -> 56
- net COL0: track 0.00 -> 46.1 mm, vias 0 -> 2
- net CRS0: track 0.00 -> 41.9 mm, vias 0 -> 2
- net NWAYEN0: track 0.00 -> 41.3 mm, vias 0 -> 2
- net /Tile0/EthernetPort0/NWAYEN: track 31.5 -> 0.00 mm, vias 2 -> 0
- net /Tile0/EthernetPort0/COL: track 30.4 -> 0.00 mm, vias 2 -> 0
- net /Tile0/EthernetPort0/CRS: track 30.4 -> 0.00 mm, vias 2 -> 0
- net (no net): track 16.5 -> 0.00 mm, vias 1 -> 0
- net Net-(C125-Pad1): track 12.1 -> 23.7 mm
- net Net-(C131-Pad1): track 9.96 -> 17.8 mm
- net /Tile0/EthernetPort1/COL: track 65.2 -> 71.6 mm
- net Net-(C121-Pad1): track 5.33 -> 10.7 mm
- net /Tile0/EthernetPort1/CRS: track 64.2 -> 69.0 mm
- net /PG_5V: track 9.73 -> 13.8 mm, vias 2 -> 3
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