File: HW/Tile0.sch (KiCad schematic (older format))
At the start: 2 parts, among them U1 XL216-512-TQ128_CHIP_VIEW

Commit message: Releasing IsoSwitch.201802
Parts:
- added J7: NWAY_TP, Measurement_Points:Measurement_Point_Square-SMD-Pad_Small, symbol TEST_1P
- added J8: CRS_TP, Measurement_Points:Measurement_Point_Square-SMD-Pad_Small, symbol TEST_1P
- added J9: COL_TP, Measurement_Points:Measurement_Point_Square-SMD-Pad_Small, symbol TEST_1P
Connections:
- net EthernetPort1/COL: now also J9.1
- net EthernetPort1/CRS: now also J8.1
- net EthernetPort1/NWAYEN: now also J7.1
- net EthernetPort0/COL renamed COL0
- net EthernetPort0/CRS renamed CRS0
- net EthernetPort0/NWAYEN renamed NWAYEN0
Changed lines of the file:
@@
 LIBS:contrib
 LIBS:valves
-LIBS:10118193-0001LF
-LIBS:615032137821
 LIBS:HW-cache
 EELAYER 25 0
@@
 P 5800 3150
 AR Path="/5A49BC89" Ref="#PWR0117"  Part="1"
-AR Path="/5A436E1B/5A49BC89" Ref="#PWR0123"  Part="1"
-F 0 "#PWR0123" H 5800 2900 50  0001 C CNN
+AR Path="/5A436E1B/5A49BC89" Ref="#PWR0125"  Part="1"
+F 0 "#PWR0125" H 5800 2900 50  0001 C CNN
 F 1 "GND" H 5800 3000 50  0000 C CNN
 F 2 "" H 5800 3150 50  0001 C CNN
@@
 $EndComp
 $Comp
-L +3V3 #PWR0124
+L +3V3 #PWR0126
 U 1 1 5A4F6830
 P 4300 7250
-F 0 "#PWR0124" H 4300 7100 50  0001 C CNN
+F 0 "#PWR0126" H 4300 7100 50  0001 C CNN
 F 1 "+3V3" H 4300 7390 50  0000 C CNN
 F 2 "" H 4300 7250 50  0001 C CNN
@@
 Text Notes 4550 7400 0    60   ~ 0
 Pull-Up to enable boot from XTAG
+$Comp
+L TEST_1P J9
+U 1 1 5A6AA219
+P 7900 750
+F 0 "J9" H 7900 1020 50  0000 C CNN
+F 1 "COL_TP" H 7900 950 50  0000 C CNN
+F 2 "Measurement_Points:Measurement_Point_Square-SMD-Pad_Small" H 8100 750 50  0001 C CNN
+F 3 "" H 8100 750 50  0001 C CNN
+	1    7900 750
+	-1   0    0    1
+$EndComp
+$Comp
+L TEST_1P J8
+U 1 1 5A6AA35A
+P 7600 850
+F 0 "J8" H 7600 1120 50  0000 C CNN
+F 1 "CRS_TP" H 7600 1050 50  0000 C CNN
+F 2 "Measurement_Points:Measurement_Point_Square-SMD-Pad_Small" H 7800 850 50  0001 C CNN
+F 3 "" H 7800 850 50  0001 C CNN
+	1    7600 850
+	-1   0    0    1
+$EndComp
+$Comp
+L TEST_1P J7
+U 1 1 5A6AE453
+P 7300 950
+F 0 "J7" H 7300 1220 50  0000 C CNN
+F 1 "NWAY_TP" H 7300 1150 50  0000 C CNN
+F 2 "Measurement_Points:Measurement_Point_Square-SMD-Pad_Small" H 7500 950 50  0001 C CNN
+F 3 "" H 7500 950 50  0001 C CNN
+	1    7300 950
+	-1   0    0    1
+$EndComp
+Connection ~ 7300 950
+Connection ~ 7600 850
+Connection ~ 7900 750
+Text GLabel 3050 6850 3    60   Input ~ 0
+NWAYEN0
+Connection ~ 3050 6850
+Connection ~ 3350 6750
+Connection ~ 3650 6650
+Text GLabel 3350 6750 3    60   Input ~ 0
+CRS0
+Text GLabel 3650 6650 3    60   Input ~ 0
+COL0
 $EndSCHEMATC
